Commit message: falta arregalar full

File: motoman_sda10f_support/urdf/environment_macro.xacro (robot description, xacro)
@@ -1,5 +1,7 @@
 <?xml version="1.0" ?>
 <model xmlns:xacro="http://ros.org/wiki/xacro">
+	<xacro:include filename="$(find motoman_sda10f_support)/urdf/zed_macro.xacro"/><!-- ZED camera -->
 	<xacro:macro name="environment" params="name prefix">
+	<xacro:zed_camera prefix=""/>
 		<!-- link list -->
 	<link name="conveyor">
@@ -52,5 +54,5 @@
 		</visual>
 </link>
-	<link name="table">
+	<!--link name="table">
 		<visual>
 			<geometry>
@@ -63,6 +65,6 @@
 			</material>
 		</visual>
-</link>
-	<link name="worktable">
+</link-->
+	<!--link name="worktable">
 		<visual>
 			<geometry>
@@ -74,4 +76,15 @@
 			</material>
 		</visual>
+</link-->
+	<link name="worktable">
+		<visual>
+			<geometry>
+				<mesh filename="package://motoman_sda10f_support/meshes/environment/table_new.stl" scale="0.001 0.001 0.001"/>
+			</geometry>
+			<origin xyz="0 0 0"/>
+			<material name="gray_conveyor">
+				<texture filename="package://motoman_sda10f_support/meshes/environment/textures/red.png"/>
+			</material>
+		</visual>
 </link>
 	<link name="beacon">
@@ -97,5 +110,5 @@
 		</visual>
 </link-->
-	<link name="mps">
+	<!--link name="mps">
 		<visual>
 			<geometry>
@@ -113,6 +126,6 @@
 				<origin xyz= "-0.7 0 -1.40"/>
 		</collision>
-</link>
-	<!--link name="MPS_FAKE">
+</link-->
+	<link name="MPS_FAKE">
 		<visual>
 			<geometry>
@@ -124,5 +137,5 @@
 			</material>
 		</visual>
-</link-->
+</link>
 		<!-- joint list -->
 	<joint name="coveyor_to_robot" type="fixed">
@@ -152,13 +165,18 @@
 		<origin xyz="1.11 0 0" rpy="0 0 0"/>
 	</joint>
-	<joint name="table_to_robot" type="fixed">
+	<!--joint name="table_to_robot" type="fixed">
 		<parent link="torso_base_link"/>
 		<child link="table"/>
-		<origin xyz="0.7 0 -0.3" rpy="1.571 0 -1.571"/>
-	</joint>
-	<joint name="worktable_to_robot" type="fixed">
+		<origin xyz="0.7 0 -0.34" rpy="1.571 0 -1.571"/>
+	</joint-->
+	<!--joint name="worktable_to_robot" type="fixed">
 		<parent link="table"/>
 		<child link="worktable"/>
 		<origin xyz="0 1.28 -0.76" rpy="0 0 0"/>
+	</joint-->
+	<joint name="worktable_to_robot" type="fixed">
+		<parent link="torso_base_link"/>
+		<child link="worktable"/>
+		<origin xyz="0.52 0 0.29" rpy="0 0  1.57"/>
 	</joint>
 	<joint name="beacon_to_robot" type="fixed">
@@ -172,14 +190,20 @@
 		<origin xyz="-0.53 -0.54 -0.3" rpy="1.571 0 1.571"/>
 	</joint-->
-		<joint name="mps_to_robot" type="fixed">
+		<!--joint name="mps_to_robot" type="fixed">
 		<parent link="torso_base_link"/>
 		<child link="mps"/>
-		<origin xyz="-0.111 -1.405 -0.3" rpy="1.571 0 1.571"/> <!--Sumo 5cm a las MPS por si acaso-->
-	</joint>
-		<!--joint name="MPS_FAKE_to_robot" type="fixed">
+		<origin xyz="-0.111 -1.405 -0.3" rpy="1.571 0 1.571"/--> <!--Sumo 5cm a las MPS por si acaso-->
+	<!--/joint-->
+	<joint name="MPS_FAKE_to_robot" type="fixed">
 		<parent link="torso_base_link"/>
 		<child link="MPS_FAKE"/>
-		<origin xyz="-1.35 0.6 -0.3" rpy="0 0 -1.5708"/--> <!--Sumo 5cm a las MPS por si acaso-->
-	<!--/joint-->
+		<origin xyz="-1.35 0.6 -0.3" rpy="0 0 -1.5708"/> <!--Sumo 5cm a las MPS por si acaso-->
+	</joint>
+	<!-- Camera zed -->
+	<joint name="zed_camera" type="fixed">
+		<parent link="torso_base_link" />
+		<child link = "zed_camera_center" />
+		<origin xyz="0 0 3" rpy="0 1.57 0" />
+	</joint>
 		<!-- end of joint list -->
 	</xacro:macro>

File: motoman_sda10f_support/urdf/sda10f_macro.xacro (robot description, xacro)
@@ -3,5 +3,4 @@
 	<xacro:include filename="$(find motoman_sda10f_support)/urdf/common_torso_macro.xacro" />
 	<xacro:include filename="$(find motoman_sda10f_support)/urdf/arm_macro.xacro" />
-	<xacro:include filename="$(find motoman_sda10f_support)/urdf/robotiq_c2_model_macro.xacro"/>
 	<xacro:include filename="$(find robotiq_s_model_visualization)/cfg/s-model_articulated_macro.xacro"/>
 	<xacro:include filename="$(find motoman_sda10f_support)/urdf/kinect_macro.xacro" />
@@ -18,30 +17,37 @@
 		</xacro:motoman_arm>
 		<!--Grippers-->
-		<xacro:robotiq_c2_model prefix=""/>
 		<xacro:s-model_articulated prefix=""/>
 		<!--Grippers with robot joints-->
-		<joint name="left_gripper_to_robot" type="fixed">
-			<parent link="${prefix}arm_left_link_tool0" />
-			<child link = "${prefix}robotiq_85_base_link" />
-			<origin xyz="0 0 -0.034" rpy="0 1.5708 2.3562" />
-		</joint>
-		<joint name="right_gripper_to_robot" type="fixed">
+       		<joint name="right_gripper_to_robot" type="fixed">
 			<parent link="${prefix}arm_right_link_tool0" />
-			<child link = "${prefix}palm" />
+			<child link ="${prefix}palm" />
 			<origin xyz="0 0 -0.065" rpy="-1.5708 0 1.5708" />
 		</joint>
-		<!--Create and update TCP pose -->
 		<link name="arm_right_tcp_link" />
 		<link name="arm_left_tcp_link" />
+		<link name="vacuum_gripper">
+			<visual>
+				<geometry>
+					<mesh filename="package://motoman_sda10f_support/meshes/environment/vacuum_gripper.stl" scale="0.001 0.001 0.001"/>
+				</geometry>
+				<origin xyz="0 0 0"/>
+				<material name="gray_conveyor"/>
+			</visual>
+		</link>
 		<!--Define the position of the TCP with respect to the arm flange-->
 		<joint name="arm_right_tool0_to_tcp" type="fixed" >
 			<parent link="${prefix}arm_right_link_tool0" />
 			<child link = "${prefix}arm_right_tcp_link" />
-			<origin xyz="0 0 -0.23" rpy="3.1416 0 0" />
+			<origin xyz="0 0 -0.23" rpy="3.1416 0 1.5708" />
 		</joint>
-		<joint name="arm_left_tool0_to_tcp" type="fixed" >
+		<joint name="vacuum_gripper" type="fixed">
 			<parent link="${prefix}arm_left_link_tool0" />
-			<child link = "${prefix}arm_left_tcp_link" />
-			<origin xyz="0 0 -0.15" rpy="3.1416 0 0.7854" />
+			<child link="vacuum_gripper"/>
+        		<origin xyz="0 0 -0.147" rpy="3.14 0 0" />
+		</joint>
+		<joint name="arm_left_vacumm_to_tcp" type="fixed" >
+			<parent link="vacuum_gripper" />
+			<child link ="${prefix}arm_left_tcp_link" />
+			<origin xyz="0 0 0" rpy="0 0 0" />
 		</joint>
 		</xacro:macro>

File: motoman_sda10f_support/urdf/simple_sda10f_macro.xacro (robot description, xacro)
@@ -3,9 +3,9 @@
      <xacro:include filename="$(find motoman_sda10f_support)/urdf/common_torso_macro.xacro" />
      <xacro:include filename="$(find motoman_sda10f_support)/urdf/arm_macro.xacro" />
-     <xacro:include filename="$(find motoman_sda10f_support)/urdf/robotiq_c2_model_macro.xacro"/>
      <xacro:include filename="$(find robotiq_s_model_visualization)/cfg/s-model_articulated_macro.xacro"/>
      <xacro:include filename="$(find motoman_sda10f_support)/urdf/kinect_macro.xacro" />
 	<xacro:include filename="$(find motoman_sda10f_support)/urdf/environment_macro.xacro"/>
 	<xacro:include filename="$(find motoman_sda10f_support)/urdf/real_sense_macro.xacro"/>
+	<!--xacro:include filename="$(find motoman_sda10f_support)/urdf/zed_macro.xacro"/--><!-- ZED camera LLAMADA EN ENVIRONMENT.XACRO OJOOOOO MODIFICAR ESTO-->
 	<!--xacro:include filename="$(find motoman_sda10f_support)/urdf/aruco_marker_macro.xacro"/-->
      <xacro:macro name="motoman_sda10f" params="prefix">
@@ -17,12 +17,7 @@
             <origin xyz="0.09996 -0.0275 0.32214" rpy="1.57 0 0" />
         </xacro:motoman_arm>
-        <xacro:robotiq_c2_model prefix=""/>
+        <!--xacro:robotiq_c2_model prefix=""/-->
 		<xacro:s-model_articulated prefix=""/>
 		<!--Grippers with robot joints-->
-		<joint name="left_gripper_to_robot" type="fixed">
-			<parent link="${prefix}arm_left_link_tool0" />
-			<child link = "${prefix}robotiq_85_base_link" />
-			<origin xyz="0 0 -0.034" rpy="0 1.5708 2.3562" />
-		</joint>
 		<joint name="right_gripper_to_robot" type="fixed">
 			<parent link="${prefix}arm_right_link_tool0" />
@@ -33,14 +28,28 @@
 		<link name="arm_right_tcp_link" />
 		<link name="arm_left_tcp_link" />
+		<link name="vacuum_gripper">
+			<visual>
+				<geometry>
+					<mesh filename="package://motoman_sda10f_support/meshes/environment/vacuum_gripper.stl" scale="0.001 0.001 0.001"/>
+				</geometry>
+				<origin xyz="0 0 0"/>
+				<material name="gray_conveyor"/>
+			</visual>
+		</link>
 		<!--Define the position of the TCP with respect to the arm flange-->
 		<joint name="arm_right_tool0_to_tcp" type="fixed" >
 			<parent link="${prefix}arm_right_link_tool0" />
 			<child link = "${prefix}arm_right_tcp_link" />
-			<origin xyz="0 0 -0.23" rpy="3.1416 0 0" />
+			<origin xyz="0 0 -0.23" rpy="3.1416 0 1.5708" />
 		</joint>
-		<joint name="arm_left_tool0_to_tcp" type="fixed" >
+		<joint name="vacuum_gripper" type="fixed">
 			<parent link="${prefix}arm_left_link_tool0" />
+			<child link="vacuum_gripper"/>
+        		<origin xyz="0 0 -0.147" rpy="3.14 0 0" />
+		</joint>
+		<joint name="arm_left_vacumm_to_tcp" type="fixed" >
+			<parent link="vacuum_gripper" />
 			<child link = "${prefix}arm_left_tcp_link" />
-			<origin xyz="0 0 -0.15" rpy="3.1416 0 0.7854" />
+			<origin xyz="0 0 0" rpy="0 0 0" />
 		</joint>
      </xacro:macro>
